File: MCU_Datalogger_KiCad/connectors.kicad_sch (KiCad schematic)
At the start: 4 parts, among them J1 Conn_01x04_Male, J2 Conn_01x04_Male, J3 Conn_01x09_Male, J4 Conn_02x03_Odd_Even

Commit message: Placement of footprints
Parts:
- J2: footprint Connector_PinHeader_2.54mm:PinHeader_1x04_P2.54mm_Horizontal -> Connector_PinHeader_2.54mm:PinHeader_1x04_P2.54mm_Vertical
Changed lines of the file:
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@@
     (property "Reference" "J2" (id 0) (at 65.405 30.48 0))
     (property "Value" "Conn_01x04_Male" (id 1) (at 65.405 33.02 0))
-    (property "Footprint" "Connector_PinHeader_2.54mm:PinHeader_1x04_P2.54mm_Horizontal" (id 2) (at 64.77 38.1 0)
+    (property "Footprint" "Connector_PinHeader_2.54mm:PinHeader_1x04_P2.54mm_Vertical" (id 2) (at 64.77 38.1 0)
       (effects (font (size 1.27 1.27)) hide)
     )
