File: MCU_Datalogger_KiCad/MCU_Datalogger_KiCad.kicad_sch (KiCad schematic)
At the start: 0 parts

Commit message: Addition of components
Parts:
- added BT?: Battery, symbol Device:Battery
- added C? (x4): C, symbol Device:C
- added C?: C_Polarized, symbol Device:C_Polarized
- added D? (x2): LED, symbol Device:LED
- added H? (x4): MountingHole, symbol Mechanical:MountingHole
- added R? (x7): R, symbol Device:R
- added U? (x2): 24LC1025, symbol Memory_EEPROM:24LC1025
- added U?: ATMEGA328P-AU, QFP80P900X900X120-32N, symbol ATMEGA328P-AU:ATMEGA328P-AU
- added U?: DS1337S+, SOIC127P600X175-8N, symbol DS1337S_:DS1337S+
- added Y? (x2): Crystal, symbol Device:Crystal
Connections:
- new net: U?.21 (GND), U?.3 (GND), U?.5 (GND)
- new net: U?.4 (VCC), U?.6 (VCC)
Other:
- added sheet Connectors (connectors.kicad_sch)

Commit message: Annotation
Parts:
- gave numbers to parts that had none: 25
Other:
- moved on the sheet: BT1, C1, C2, C3, C4, C5, D1, D2, H1, H2, H3, H4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

Commit message: Values of components
Parts:
- C1, C4: value C -> 0.1uF
- C2, C3: value C -> 22pF
- C5: value C_Polarized -> 100nF
- R1, R3: value R -> 4.7k
- R2, R4: value R -> 10K
- R5, R7: value R -> 330
- R6: value R -> 10k
- Y1: value Crystal -> 32.768 KHz
- Y2: value Crystal -> 16 MHz
Changed lines of the file:
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@@
     (in_bom yes) (on_board yes) (fields_autoplaced)
     (property "Reference" "R5" (id 0) (at 144.78 33.02 90))
-    (property "Value" "R" (id 1) (at 144.78 35.56 90))
+    (property "Value" "330" (id 1) (at 144.78 35.56 90))
     (property "Footprint" "" (id 2) (at 144.78 41.148 90)
       (effects (font (size 1.27 1.27)) hide)
@@
       (effects (font (size 1.27 1.27)) (justify left))
     )
-    (property "Value" "R" (id 1) (at 87.63 167.6399 0)
+    (property "Value" "4.7k" (id 1) (at 87.63 167.6399 0)
       (effects (font (size 1.27 1.27)) (justify left))
     )
@@
       (effects (font (size 1.27 1.27)) (justify left))
     )
-    (property "Value" "R" (id 1) (at 104.14 38.0999 0)
+    (property "Value" "10K" (id 1) (at 104.14 38.0999 0)
       (effects (font (size 1.27 1.27)) (justify left))
     )
@@
     (in_bom yes) (on_board yes) (fields_autoplaced)
     (property "Reference" "R6" (id 0) (at 160.02 73.66 90))
-    (property "Value" "R" (id 1) (at 160.02 76.2 90))
+    (property "Value" "10k" (id 1) (at 160.02 76.2 90))
     (property "Footprint" "" (id 2) (at 160.02 81.788 90)
       (effects (font (size 1.27 1.27)) hide)
@@
       (effects (font (size 1.27 1.27)) (justify left))
     )
-    (property "Value" "R" (id 1) (at 232.41 67.3099 0)
+    (property "Value" "330" (id 1) (at 232.41 67.3099 0)
       (effects (font (size 1.27 1.27)) (justify left))
     )
@@
       (effects (font (size 1.27 1.27)) (justify left))
     )
-    (property "Value" "C" (id 1) (at 148.59 72.3899 0)
+    (property "Value" "22pF" (id 1) (at 148.59 72.3899 0)
       (effects (font (size 1.27 1.27)) (justify left))
     )
@@
       (effects (font (size 1.27 1.27)) (justify left))
     )
-    (property "Value" "R" (id 1) (at 95.25 38.0999 0)
+    (property "Value" "10K" (id 1) (at 95.25 38.0999 0)
       (effects (font (size 1.27 1.27)) (justify left))
     )
@@
       (effects (font (size 1.27 1.27)) (justify left))
     )
-    (property "Value" "C" (id 1) (at 148.59 59.6899 0)
+    (property "Value" "22pF" (id 1) (at 148.59 59.6899 0)
       (effects (font (size 1.27 1.27)) (justify left))
     )
@@
       (effects (font (size 1.27 1.27)) (justify left))
     )
-    (property "Value" "C" (id 1) (at 116.84 38.0999 0)
+    (property "Value" "0.1uF" (id 1) (at 116.84 38.0999 0)
       (effects (font (size 1.27 1.27)) (justify left))
     )
@@
     (in_bom yes) (on_board yes) (fields_autoplaced)
     (property "Reference" "Y1" (id 0) (at 33.02 38.1 0))
-    (property "Value" "Crystal" (id 1) (at 33.02 40.64 0))
+    (property "Value" "32.768 KHz" (id 1) (at 33.02 40.64 0))
     (property "Footprint" "" (id 2) (at 33.02 45.72 0)
       (effects (font (size 1.27 1.27)) hide)
@@
     (in_bom yes) (on_board yes) (fields_autoplaced)
     (property "Reference" "C4" (id 0) (at 158.75 16.51 90))
-    (property "Value" "C" (id 1) (at 158.75 19.05 90))
+    (property "Value" "0.1uF" (id 1) (at 158.75 19.05 90))
     (property "Footprint" "" (id 2) (at 162.56 23.1648 0)
       (effects (font (size 1.27 1.27)) hide)
@@
       (effects (font (size 1.27 1.27)) (justify right))
     )
-    (property "Value" "Crystal" (id 1) (at 162.56 57.1499 90)
+    (property "Value" "16 MHz" (id 1) (at 162.56 57.1499 90)
       (effects (font (size 1.27 1.27)) (justify right))
     )
@@
       (effects (font (size 1.27 1.27)) (justify left))
     )
-    (property "Value" "R" (id 1) (at 96.52 167.6399 0)
+    (property "Value" "4.7k" (id 1) (at 96.52 167.6399 0)
       (effects (font (size 1.27 1.27)) (justify left))
     )
@@
       (effects (font (size 1.27 1.27)) (justify left))
     )
-    (property "Value" "C_Polarized" (id 1) (at 233.68 34.6709 0)
+    (property "Value" "100nF" (id 1) (at 233.68 34.6709 0)
       (effects (font (size 1.27 1.27)) (justify left))
     )
@@
     )
     (path "/b746dac3-e803-4265-b4d7-618e18587818"
-      (reference "C1") (unit 1) (value "C") (footprint "")
+      (reference "C1") (unit 1) (value "0.1uF") (footprint "")
     )
     (path "/a7fecb47-a0a4-48a1-bace-88c19aa5da0d"
-      (reference "C2") (unit 1) (value "C") (footprint "")
+      (reference "C2") (unit 1) (value "22pF") (footprint "")
     )
     (path "/9a0d6194-b880-4cd8-b73f-18323b8c24a3"
-      (reference "C3") (unit 1) (value "C") (footprint "")
+      (reference "C3") (unit 1) (value "22pF") (footprint "")
     )
     (path "/e5fe5a19-ca5b-43e3-b01a-d52c6f069d36"
-      (reference "C4") (unit 1) (value "C") (footprint "")
+      (reference "C4") (unit 1) (value "0.1uF") (footprint "")
     )
     (path "/fbced520-6da2-4de5-ab80-539bd423e428"
-      (reference "C5") (unit 1) (value "C_Polarized") (footprint "")
+      (reference "C5") (unit 1) (value "100nF") (footprint "")
     )
     (path "/78903299-8531-4ae9-a09c-a7daabf2d597"
@@
     )
     (path "/16dd5ee8-835d-4394-8b0e-be59852f7d3a"
-      (reference "R1") (unit 1) (value "R") (footprint "")
+      (reference "R1") (unit 1) (value "4.7k") (footprint "")
     )
     (path "/a3667980-12eb-41f3-be57-62da8259e1ed"
-      (reference "R2") (unit 1) (value "R") (footprint "")
+      (reference "R2") (unit 1) (value "10K") (footprint "")
     )
     (path "/f34101b6-4aac-4c3d-93ac-cf78ab254faa"
-      (reference "R3") (unit 1) (value "R") (footprint "")
+      (reference "R3") (unit 1) (value "4.7k") (footprint "")
     )
     (path "/5b57aefb-76bd-4b4d-96d4-ede072d6b2f0"
-      (reference "R4") (unit 1) (value "R") (footprint "")
+      (reference "R4") (unit 1) (value "10K") (footprint "")
     )
     (path "/03145d1a-5990-4aab-a87e-654e43289dd0"
-      (reference "R5") (unit 1) (value "R") (footprint "")
+      (reference "R5") (unit 1) (value "330") (footprint "")
     )
     (path "/6be3a39c-7b64-4eb6-8c8c-bab2d2913b37"
-      (reference "R6") (unit 1) (value "R") (footprint "")
+      (reference "R6") (unit 1) (value "10k") (footprint "")
     )
     (path "/933ab64c-547b-49a3-89bb-1daace63ef41"
-      (reference "R7") (unit 1) (value "R") (footprint "")
+      (reference "R7") (unit 1) (value "330") (footprint "")
     )
     (path "/3a133edd-713b-401a-ac1a-d7c8459232c7"
@@
     )
     (path "/dafe4851-5277-4940-88ca-da4c1af048d9"
-      (reference "Y1") (unit 1) (value "Crystal") (footprint "")
+      (reference "Y1") (unit 1) (value "32.768 KHz") (footprint "")
     )
     (path "/ef523510-ad1b-49cc-8946-87884bcd5ed2"
-      (reference "Y2") (unit 1) (value "Crystal") (footprint "")
-    )
-  )
+      (reference "Y2") (unit 1) (value "16 MHz") (footprint "")
+    )
+  )

Commit message: Footprint association
Parts:
- BT1: footprint (none) -> Connector_PinHeader_2.54mm:PinHeader_1x02_P2.54mm_Vertical
- C1, C2, C3, C4, C5: footprint (none) -> Capacitor_SMD:C_0805_2012Metric
- D1, D2: footprint (none) -> LED_SMD:LED_0805_2012Metric
- H1, H2, H3, H4: footprint (none) -> MountingHole:MountingHole_2.1mm
- R1, R2, R3, R4, R5, R6, R7: footprint (none) -> Resistor_SMD:R_0805_2012Metric
- U1, U3: footprint (none) -> Package_SO:SOIC-8_5.23x5.23mm_P1.27mm
- U2: footprint SOIC127P600X175-8N -> DS1337S_:SOIC127P600X175-8N
- U4: footprint QFP80P900X900X120-32N -> ATMEGA328P-AU:QFP80P900X900X120-32N
- Y1, Y2: footprint (none) -> Crystal:Crystal_SMD_5032-2Pin_5.0x3.2mm_HandSoldering

Commit message: WIRING sheet 1
Connections:
- net at BT1.1 (+): now also C5.1, D2.2 (A), U4.18 (AVCC), U4.4 (VCC)
- net GND: now reaches BT1.2 (-)
- net GND: now also C1.2, C2.1, C3.1, C4.1, C5.2, R5.1, R7.2, U1.4 (GND), U1.7 (WP), U2.4 (GND), U3.2 (A1), U3.4 (GND), U3.7 (WP), U4.21 (GND), U4.3 (GND), U4.5 (GND)
- net at R5.2: now also D1.1 (K)
- net Vcc: now reaches R1.1
- net Vcc: now also C1.1, R2.1, R3.1, R4.1, R6.1, U1.1 (A0), U1.2 (A1), U1.3 (A2), U1.8 (VCC), U2.8 (VCC), U3.1 (A0), U3.3 (A2), U3.8 (VCC)
- net SCK: now reaches R1.2
- net SCK: now also U1.6 (SCL), U2.6 (SCL), U3.6 (SCL), U4.28 (PC5)
- net SDA: now reaches U1.5 (SDA)
- net SDA: now also R3.2, U2.5 (SDA), U3.5 (SDA), U4.27 (PC4)
- net D3: now reaches U4.1 (PD3)
- net D6: now reaches U4.10 (PD6)
- net D7: now reaches U4.11 (PD7)
- net D8: now reaches U4.12 (PB0)
- net MOSI: now reaches U4.15 (PB3)
- net MISO: now reaches U4.16 (PB4)
- net SDK: now reaches U4.17 (PB5)
- net SDK: now also D1.2 (A)
- net D4: now reaches U4.2 (PD4)
- net at U4.20 (AREF): now also C4.2
- net at U4.29 (PC6/~{RESET}): now also R6.2
- net RX: now reaches U4.30 (PD0)
- net TX: now reaches U4.31 (PD1)
- net D2: now reaches U4.32 (PD2)
- net at U4.6 (VCC): no longer U4.4 (VCC)
- net at U4.7 (PB6): now also C2.2, Y2.2
- net at U4.8 (PB7): now also C3.2, Y2.1
- net D5: now reaches U4.9 (PD5)
- net at R4.2: now also U2.7 (SQW/~INT)
- net at R7.1: now also D2.1 (K)
- net at R2.2: now also U2.3 (~{INTA})
- net at U2.1 (X1): now also Y1.1
- net at U2.2 (X2): now also Y1.2
- no-connect marks 0 -> 9
Other:
- moved on the sheet: BT1, C2, C3, C4, C5, D1, D2, R1, R3, R5, R6, R7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

Commit message: Wiring sheet 2
Connections:
- net RESET: now reaches R6.2, U4.29 (PC6/~{RESET})
Other:
- sheet Connectors ports: added D2, D3, D4, D5, D6, D7, D8, GND, MISO, MOSI, RESET, RX, SCK, SDA, TX, Vcc; removed none

Commit message: Completed comments
Other:
- note added: "EEPROM"
- note added: "MCU"
- note added: "Real time clock"
- moved on the sheet: C1, H1, H2, H3, H4, R2, R4, U2, Y1
