File: MCU_Datalogger_KiCad/MCU_Datalogger_KiCad.kicad_sch (KiCad schematic)
At the start: 25 parts, among them U1 24LC1025, U2 DS1337S+, U3 24LC1025, U4 ATMEGA328P-AU, Y1 32.768 KHz, Y2 16 MHz

Commit message: Routing
Connections:
- net SDK is gone; now on net SCK: D1.2 (A), U4.17 (PB5)
Changed lines of the file:
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@@
     (effects (font (size 1.27 1.27)) (justify right bottom))
   )
-  (label "SDK" (at 193.04 59.69 180)
+  (label "SCK" (at 193.04 59.69 180)
     (effects (font (size 1.27 1.27)) (justify right bottom))
   )
