File: MCU_Datalogger_KiCad/MCU_Datalogger_KiCad.kicad_pcb (KiCad board)
At the start: 2 copper layers, 47 x 32.8 mm, 29 parts, among them J1 Conn_01x04_Male, J2 Conn_01x04_Male, J3 Conn_01x09_Male, J4 Conn_02x03_Odd_Even, U1 24LC1025, U2 DS1337S+, U3 24LC1025, U4 ATMEGA328P-AU, Y1 32.768 KHz, Y2 16 MHz

Commit message: Started but didn't finish the routing
Parts:
- moved C2 5.08 mm to (62.5, 54.9)
- moved C4 5.08 mm to (62.6, 57.7)
- moved R1 2.33 mm to (58.3, 51.3)
- moved R3 2.33 mm to (58.3, 48.8)
- moved Y2 1.90 mm to (50.8, 59.7)
- moved R6 1.24 mm to (62.9, 49.8)
- moved R5 0.44 mm to (58.5, 45.7)
- moved U4 0.25 mm to (49.8, 50.8)
- moved U1 0.13 mm to (38.6, 52.1)
Routing:
- net GND: track 111.0 -> 12.7 mm, vias 8 -> 0
- net /Vcc: track 100.3 -> 9.60 mm, vias 2 -> 0
- net /SCK: track 83.6 -> 18.9 mm, vias 7 -> 0
- net Net-(BT1-Pad1): track 54.3 -> 0.00 mm, vias 2 -> 0
- net /SDA: track 55.6 -> 17.4 mm, vias 5 -> 0
- net Net-(C3-Pad2): track 29.2 -> 0.00 mm, vias 2 -> 0
- net /D2: track 26.7 -> 0.00 mm, vias 1 -> 0
- net /MOSI: track 26.4 -> 0.00 mm
- net /RESET: track 23.0 -> 0.00 mm, vias 2 -> 0
- net Net-(C2-Pad2): track 22.6 -> 0.00 mm
- net /MISO: track 19.9 -> 0.00 mm, vias 2 -> 0
- net Net-(C4-Pad2): track 13.0 -> 0.00 mm, vias 2 -> 0
- net Net-(D2-Pad1): track 5.72 -> 0.00 mm, vias 2 -> 0
- net /D8: track 12.0 -> 16.7 mm, vias 1 -> 0
- net Net-(D1-Pad1): track 3.85 -> 0.00 mm
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- removed copper zone on F.Cu, net /Vcc
- removed copper zone on B.Cu, net GND
Other:
- copper layers 2 -> 4
